Commit message: downdraft table setup added

File: urdf/macros/_common.urdf.xacro (robot description, xacro)
@@ -6,3 +6,27 @@
     </material>
   </xacro:macro>  <!-- trossen_black -->
+  <material name="grey">
+        <color rgba="0.2 0.2 0.2 1.0" />
+    </material>
+    <material name="light_grey">
+        <color rgba="0.75 0.75 0.7 1" />
+    </material>
+    <material name="pink">
+        <color rgba="1.0 0.71 0.76 1.0"/>
+    </material>
+    <material name="blue">
+        <color rgba="0.1 0.2 0.6 1.0"/>
+    </material>
+    <material name="light_blue">
+        <color rgba="0.3 0.45 0.78 1.0"/>
+    </material>
+    <material name="green">
+        <color rgba="0.0 0.5 0.0 1.0" />
+    </material>
+    <material name="orange">
+        <color rgba="1.0 0.5 0.0 1.0" />
+    </material>
+    <material name="blue_green">
+        <color rgba="0.0 0.7 0.7 1.0" />
+    </material>
 </robot>

File: urdf/macros/_wxai.ros2_control.xacro (robot description, xacro)
@@ -1,5 +1,5 @@
 <?xml version="1.0"?>
 <robot xmlns:xacro="http://www.ros.org/wiki/xacro">
-  <xacro:macro name="ros2_control_joint" params="name">
+  <xacro:macro name="ros2_control_joint" params="name initial_value:=0.0">
     <joint name="${name}">
       <command_interface name="position" />
@@ -7,5 +7,5 @@
       <command_interface name="external_effort" />
       <state_interface name="position">
-        <param name="initial_value">0.0</param>
+        <param name="initial_value">${initial_value}</param>
       </state_interface>
       <state_interface name="velocity">
@@ -30,10 +30,10 @@
         </xacro:if>  <!-- ros2_control_hardware_type == 'real' -->
       </hardware>
-      <xacro:ros2_control_joint name="${prefix}joint_0"/>
-      <xacro:ros2_control_joint name="${prefix}joint_1"/>
-      <xacro:ros2_control_joint name="${prefix}joint_2"/>
-      <xacro:ros2_control_joint name="${prefix}joint_3"/>
-      <xacro:ros2_control_joint name="${prefix}joint_4"/>
-      <xacro:ros2_control_joint name="${prefix}joint_5"/>
+      <xacro:ros2_control_joint name="${prefix}joint_0" initial_value="0.0"/>
+      <xacro:ros2_control_joint name="${prefix}joint_1" initial_value="0.8"/>
+      <xacro:ros2_control_joint name="${prefix}joint_2" initial_value="0.8"/>
+      <xacro:ros2_control_joint name="${prefix}joint_3" initial_value="0.0"/>
+      <xacro:ros2_control_joint name="${prefix}joint_4" initial_value="0.0"/>
+      <xacro:ros2_control_joint name="${prefix}joint_5" initial_value="0.0"/>
       <joint name="${prefix}left_carriage_joint">
         <command_interface name="position" />

File: urdf/wxai.urdf.xacro (robot description, xacro)
@@ -8,4 +8,10 @@
   <xacro:arg name="ip_address"                      default="192.168.1.2"/>
   <xacro:arg name="base_link_frame"                 default="base_link"/>
+  <xacro:arg name="use_suction_cup"                 default="true"/>
+  <xacro:arg name="use_downdraft"                   default="true"/>
+  <xacro:arg name="xyz"                             default="0.75 -0.134 0.99"/>
+  <xacro:arg name="rpy"                             default="0 0 1.57"/>
+  <xacro:arg name="custom_mount_xyz"                default="-0.029 0.0 -0.02"/>
+  <xacro:arg name="custom_mount_rpy"                default="0 0 0"/>
   <xacro:if value="$(arg use_world_frame)">
     <link name="world"/>
@@ -19,10 +25,40 @@
   <xacro:include filename="$(find trossen_arm_description)/urdf/macros/_wxai.urdf.xacro" />
   <xacro:include filename="$(find trossen_arm_description)/urdf/macros/_common.urdf.xacro" />
+  <xacro:include filename="$(find trossen_arm_description)/urdf/custom_mount.xacro" />
   <xacro:trossen_black/>
   <xacro:wxai
-    variant="$(arg variant)"
-    arm_side="$(arg arm_side)"
-    prefix="$(arg prefix)"
-    ros2_control_hardware_type="$(arg ros2_control_hardware_type)"
-    ip_address="$(arg ip_address)"/>
+      variant="$(arg variant)"
+      arm_side="$(arg arm_side)"
+      prefix="$(arg prefix)"
+      ros2_control_hardware_type="$(arg ros2_control_hardware_type)"
+      ip_address="$(arg ip_address)"/>
+  <xacro:if value="$(arg use_downdraft)">
+    <xacro:include filename="$(find trossen_arm_description)/urdf/downdraft.xacro" />
+    <joint name="$(arg prefix)table_to_arm" type="fixed">
+      <parent link="$(arg prefix)Bottom_Box"/>
+      <child link="$(arg prefix)base_link"/>
+      <origin xyz="$(arg xyz)" rpy="$(arg rpy)"/>
+    </joint>
+  </xacro:if>
+  <xacro:unless value="$(arg use_downdraft)">
+    <link name="world"/>
+    <joint name="$(arg prefix)world_to_arm" type="fixed">
+        <parent link="world"/>
+        <child link="$(arg prefix)base_link"/>
+        <origin xyz="$(arg xyz)" rpy="$(arg rpy)"/>
+    </joint>
+  </xacro:unless>
+  <xacro:if value="$(arg use_suction_cup)">
+    <xacro:include filename="$(find trossen_arm_description)/urdf/suction_cup.xacro" />
+    <joint name="$(arg prefix)base_and_suction" type="fixed">
+      <parent link="$(arg prefix)link_6" />
+      <child link="$(arg prefix)base_mount" />
+      <origin xyz="0.0613 0 -0.028" rpy="0 ${pi} 0" />
+    </joint>
+  </xacro:if>
+  <joint name="$(arg prefix)custom_mount_gripper" type="fixed">
+    <parent link="$(arg prefix)link_6" />
+    <child link="$(arg prefix)Custom_Mount" />
+    <origin xyz="$(arg custom_mount_xyz)" rpy="$(arg custom_mount_rpy)" />
+  </joint>
 </robot>
