Commit message: fixed meshes

File: urdf/macros/_common.urdf.xacro (robot description, xacro)
@@ -11,3 +11,12 @@
     </material>
   </xacro:macro>  <!-- maple_tabletop -->
+  <material name="white">
+    <color rgba="1.0 1.0 1.0 1.0"/>
+  </material>
+  <material name="gold">
+    <color rgba="1.0 0.88 0.35 1.0"/>
+  </material>
+  <material name="silver">
+    <color rgba="0.753 0.753 0.753 1.0"/>
+  </material>
 </robot>

File: urdf/wxai.urdf.xacro (robot description, xacro)
@@ -8,4 +8,5 @@
   <xacro:arg name="ip_address"                      default="192.168.1.2"/>
   <xacro:arg name="base_link_frame"                 default="base_link"/>
+  <xacro:arg name="use_suction_cup"                 default="true"/>
   <xacro:if value="$(arg use_world_frame)">
     <link name="world"/>
@@ -26,3 +27,11 @@
     ros2_control_hardware_type="$(arg ros2_control_hardware_type)"
     ip_address="$(arg ip_address)"/>
+  <xacro:if value="$(arg use_suction_cup)">
+    <xacro:include filename="$(find trossen_arm_description)/urdf/suction_cup.xacro" />
+    <joint name="$(arg prefix)robot_mount_and_link_6" type="fixed">
+      <parent link="$(arg prefix)link_6" />
+      <child link="$(arg prefix)Robot_Mount" />
+      <origin xyz="0.01 0 -0.028" rpy="0 ${pi} ${pi}" />
+    </joint>
+  </xacro:if>
 </robot>
