Commit message: adjusted suction cup coordinates

File: urdf/suction_cup.xacro (robot description, xacro)
@@ -32,5 +32,5 @@
                 <mesh filename="package://trossen_arm_description/meshes/custom/suction_mount.stl" scale="0.001 0.001 0.001" />
             </geometry>
-            <material name="trossen_black"/>
+            <material name="black"/>
         </visual>
         <collision name="suction_mount_collision">
@@ -43,10 +43,10 @@
     <link name="$(arg prefix)suction_cup">
         <inertial>
-            <origin xyz="-7.315320663647534e-14 -0.030944834484754304 4.2957051116232495e-09" rpy="0.0 -0.0 0.0" />
+            <origin xyz="-7.316695537418065e-14 -0.006944834484754301 4.2957051027414655e-09" rpy="0.0 -0.0 0.0" />
             <mass value="0.009782061269685442" />
-            <inertia ixx="5.885335742899806e-06" iyy="8.570586221259282e-07" izz="5.885335740427175e-06" ixy="2.3271680856798765e-17" iyz="-4.086086937554745e-18" ixz="5.939692711156479e-22" />
+            <inertia ixx="5.885335742899833e-06" iyy="8.570586221259291e-07" izz="5.885335740427188e-06" ixy="2.327168085679879e-17" iyz="-4.086086937554745e-18" ixz="5.939692711218109e-22" />
         </inertial>
         <visual name="suction_cup_visual">
-            <origin xyz="2.016732274611434e-16 -0.060999999999999915 4.295695976708203e-09" rpy="6.488633748503318e-16 -1.5707963267948803 0" />
+            <origin xyz="1.879244897558544e-16 -0.036999999999999915 4.295695958944634e-09" rpy="6.48863374850338e-16 -1.5707963267948803 0" />
             <geometry>
                 <mesh filename="package://trossen_arm_description/meshes/custom/suction_cup.stl" scale="0.001 0.001 0.001" />
@@ -55,5 +55,5 @@
         </visual>
         <collision name="suction_cup_collision">
-            <origin xyz="2.016732274611434e-16 -0.060999999999999915 4.295695976708203e-09" rpy="6.488633748503318e-16 -1.5707963267948803 0" />
+            <origin xyz="1.879244897558544e-16 -0.036999999999999915 4.295695958944634e-09" rpy="6.48863374850338e-16 -1.5707963267948803 0" />
             <geometry>
                 <mesh filename="package://trossen_arm_description/meshes/custom/suction_cup.stl" scale="0.001 0.001 0.001" />
@@ -63,10 +63,10 @@
     <link name="$(arg prefix)tube">
         <inertial>
-            <origin xyz="2.0371946687298745e-09 -0.00521836787395407 0.010107808682448339" rpy="0.0 -0.0 0.0" />
+            <origin xyz="2.0371946549811372e-09 -0.005218367873954089 0.010107808682448321" rpy="0.0 -0.0 0.0" />
             <mass value="0.001682506141360719" />
-            <inertia ixx="1.0232240623866935e-07" iyy="5.010492163195446e-08" izz="7.051264882387267e-08" ixy="-3.457129761388185e-15" iyz="2.7203670518921504e-08" ixz="3.849352836359212e-15" />
+            <inertia ixx="1.0232240623866935e-07" iyy="5.010492163195494e-08" izz="7.051264882387267e-08" ixy="-3.457129761388185e-15" iyz="2.7203670518921504e-08" ixz="3.849352836359212e-15" />
         </inertial>
         <visual name="tube_visual">
-            <origin xyz="1.4648287464380052e-16 -4.295695958944634e-09 -0.0027999999999999137" rpy="1.6434538990973007e-16 -3.7012411737996247e-16 -1.5707963267948806" />
+            <origin xyz="1.327341369385115e-16 -4.295695972267311e-09 -0.0027999999999999314" rpy="1.643453899097362e-16 1.0247773124873877e-17 -1.5707963267948806" />
             <geometry>
                 <mesh filename="package://trossen_arm_description/meshes/custom/tube.stl" scale="0.001 0.001 0.001" />
@@ -75,5 +75,5 @@
         </visual>
         <collision name="tube_collision">
-            <origin xyz="1.4648287464380052e-16 -4.295695958944634e-09 -0.0027999999999999137" rpy="1.6434538990973007e-16 -3.7012411737996247e-16 -1.5707963267948806" />
+            <origin xyz="1.327341369385115e-16 -4.295695972267311e-09 -0.0027999999999999314" rpy="1.643453899097362e-16 1.0247773124873877e-17 -1.5707963267948806" />
             <geometry>
                 <mesh filename="package://trossen_arm_description/meshes/custom/tube.stl" scale="0.001 0.001 0.001" />
@@ -167,5 +167,5 @@
     </joint>
     <joint name="$(arg prefix)tube_and_suction_cup" type="fixed">
-        <origin xyz="0.0 0.0245 0.0" rpy="-1.5707963267948966 -0.0 0.0" />
+        <origin xyz="0.0 0.048499999999999995 0.0" rpy="-1.5707963267948966 -0.0 0.0" />
         <parent link="$(arg prefix)suction_cup" />
         <child link="$(arg prefix)tube" />

Commit message: edited suction cup coordinates

File: urdf/suction_cup.xacro (robot description, xacro)
@@ -32,5 +32,5 @@
                 <mesh filename="package://trossen_arm_description/meshes/custom/suction_mount.stl" scale="0.001 0.001 0.001" />
             </geometry>
-            <material name="black"/>
+            <material name="trossen_black"/>
         </visual>
         <collision name="suction_mount_collision">
