Commit message: changed mail cutter coordinates

File: urdf/downdraft_old.xacro (robot description, xacro)
@@ -303,10 +303,10 @@
     <link name="$(arg prefix)Mail_Spreader_Housing">
         <inertial>
-            <origin xyz="0.2297487853588787 -0.09297671857199007 0.07359079941501165" rpy="0.0 -4.663963129396153e-77 0.0" />
+            <origin xyz="0.07474878535887866 -0.0929767185719902 0.07359079941501208" rpy="0.0 -4.663963129396153e-77 0.0" />
             <mass value="0.7818877668805357" />
-            <inertia ixx="0.003421827232823249" iyy="0.004391842901898424" izz="0.0033633324964867928" ixy="-8.893594203029931e-07" iyz="2.2033683713118535e-06" ixz="-9.834189106466829e-06" />
+            <inertia ixx="0.003421827232823027" iyy="0.004391842901898535" izz="0.0033633324964865707" ixy="-8.893594203168709e-07" iyz="2.2033683713118535e-06" ixz="-9.83418910645295e-06" />
         </inertial>
         <visual name="Mail_Spreader_Housing_visual">
-            <origin xyz="0.23000000000000104 -0.10000000000000085 0.07500000000000015" rpy="-3.141592653589793 -1.5707963267948915 0" />
+            <origin xyz="0.07500000000000102 -0.10000000000000099 0.07500000000000057" rpy="-3.141592653589793 -1.5707963267948915 0" />
             <geometry>
                 <mesh filename="package://trossen_arm_description/meshes/downdraft/Mail_Spreader_Housing.stl" scale="0.001 0.001 0.001" />
@@ -315,5 +315,5 @@
         </visual>
         <collision name="Mail_Spreader_Housing_collision">
-            <origin xyz="0.23000000000000104 -0.10000000000000085 0.07500000000000015" rpy="-3.141592653589793 -1.5707963267948915 0" />
+            <origin xyz="0.07500000000000102 -0.10000000000000099 0.07500000000000057" rpy="-3.141592653589793 -1.5707963267948915 0" />
             <geometry>
                 <mesh filename="package://trossen_arm_description/meshes/downdraft/Mail_Spreader_Housing.stl" scale="0.001 0.001 0.001" />
@@ -323,10 +323,10 @@
     <link name="$(arg prefix)Mail_Top_Plate">
         <inertial>
-            <origin xyz="3.258106006185813e-05 0.07820551417803287 1.0658141036401502e-15" rpy="-2.8486550277461034e-64 -0.0 0.0" />
+            <origin xyz="3.258106006185813e-05 0.0782055141780333 1.056932319443149e-15" rpy="-2.8486550277462006e-64 -0.0 0.0" />
             <mass value="0.08915200000000002" />
-            <inertia ixx="0.0003873164201692175" iyy="0.0002032497645628878" izz="0.00018581264713210532" ixy="-1.370908783160374e-06" iyz="1.3738562485522464e-35" ixz="1.4022694188954473e-36" />
+            <inertia ixx="0.0003873164201692175" iyy="0.00020324976456292942" izz="0.00018581264713213308" ixy="-1.370908783160374e-06" iyz="-1.7347234759768069e-18" ixz="1.734723475976807e-18" />
         </inertial>
         <visual name="Mail_Top_Plate_visual">
-            <origin xyz="-2.842170943040401e-16 0.07499999999999986 1.0302869668521452e-15" rpy="-3.141592653589793 -4.857225732735152e-16 -1.5707963267948915" />
+            <origin xyz="-4.263256414560601e-16 0.07500000000000029 1.0302869668521452e-15" rpy="-3.141592653589793 -4.857225732735152e-16 -1.5707963267948915" />
             <geometry>
                 <mesh filename="package://trossen_arm_description/meshes/downdraft/Mail_Top_Plate.stl" scale="0.001 0.001 0.001" />
@@ -335,5 +335,5 @@
         </visual>
         <collision name="Mail_Top_Plate_collision">
-            <origin xyz="-2.842170943040401e-16 0.07499999999999986 1.0302869668521452e-15" rpy="-3.141592653589793 -4.857225732735152e-16 -1.5707963267948915" />
+            <origin xyz="-4.263256414560601e-16 0.07500000000000029 1.0302869668521452e-15" rpy="-3.141592653589793 -4.857225732735152e-16 -1.5707963267948915" />
             <geometry>
                 <mesh filename="package://trossen_arm_description/meshes/downdraft/Mail_Top_Plate.stl" scale="0.001 0.001 0.001" />
@@ -343,10 +343,10 @@
     <link name="$(arg prefix)Letter_Trimmer_Holder">
         <inertial>
-            <origin xyz="0.028766362717210114 -0.019520905574119354 -1.7763568394002506e-16" rpy="2.8486550277461034e-64 -0.0 0.0" />
+            <origin xyz="0.0287663627172104 -0.01952090557411964 -1.9539925233402755e-16" rpy="2.8486550277462006e-64 -0.0 0.0" />
             <mass value="0.041840657300680255" />
-            <inertia ixx="4.5702849910761456e-05" iyy="7.059497852655167e-05" izz="3.356023542885889e-05" ixy="-2.2850515949621175e-06" iyz="-1.734723475976807e-18" ixz="-1.734723475976807e-18" />
+            <inertia ixx="4.5702849910761456e-05" iyy="7.059497852653779e-05" izz="3.356023542883113e-05" ixy="-2.285051594941301e-06" iyz="4.3368086899420173e-19" ixz="-4.336808689942018e-19" />
         </inertial>
         <visual name="Letter_Trimmer_Holder_visual">
-            <origin xyz="0.034500000000000454 -0.0280000000000004 1.1723955140041654e-15" rpy="5.208585445482766e-15 -1.5707963267948961 0" />
+            <origin xyz="0.0345000000000006 -0.028000000000000684 1.1546319456101628e-15" rpy="5.208585445482771e-15 -1.5707963267948961 0" />
             <geometry>
                 <mesh filename="package://trossen_arm_description/meshes/downdraft/Letter_Trimmer_Holder.stl" scale="0.001 0.001 0.001" />
@@ -355,5 +355,5 @@
         </visual>
         <collision name="Letter_Trimmer_Holder_collision">
-            <origin xyz="0.034500000000000454 -0.0280000000000004 1.1723955140041654e-15" rpy="5.208585445482766e-15 -1.5707963267948961 0" />
+            <origin xyz="0.0345000000000006 -0.028000000000000684 1.1546319456101628e-15" rpy="5.208585445482771e-15 -1.5707963267948961 0" />
             <geometry>
                 <mesh filename="package://trossen_arm_description/meshes/downdraft/Letter_Trimmer_Holder.stl" scale="0.001 0.001 0.001" />
@@ -421,100 +421,100 @@
         </collision>
     </link>
-    <joint name="Chute_Right_and_Chute_House" type="fixed">
+    <joint name="$(arg prefix)Chute_Right_and_Chute_House" type="fixed">
         <origin xyz="-0.26322 0.0019999999999998864 -0.17350000000000002" rpy="3.141592653589793 -2.465190328815662e-32 -1.5707963267948966" />
         <parent link="$(arg prefix)Chute_01" />
         <child link="$(arg prefix)Chute_02" />
     </joint>
-    <joint name="Chute_Front_and_Chute_House" type="fixed">
+    <joint name="$(arg prefix)Chute_Front_and_Chute_House" type="fixed">
         <origin xyz="-0.0864698 0.0019999999999998864 -0.0015000000000000002" rpy="-3.141592653589793 1.3670076544845265e-15 -3.141592653589793" />
         <parent link="$(arg prefix)Chute_01" />
         <child link="$(arg prefix)Chute_03" />
     </joint>
-    <joint name="Rear_Panel_and_Top_Panel" type="fixed">
+    <joint name="$(arg prefix)Rear_Panel_and_Top_Panel" type="fixed">
         <origin xyz="0.5770000000000001 0.34880000000000005 0.0015000000000000568" rpy="1.5707963267948966 2.552890093070388e-31 0.0" />
         <parent link="$(arg prefix)Top_Panel" />
         <child link="$(arg prefix)Rear_Panel" />
     </joint>
-    <joint name="Top_Weld_Plate_and_Rear_Panel" type="fixed">
+    <joint name="$(arg prefix)Top_Weld_Plate_and_Rear_Panel" type="fixed">
         <origin xyz="-0.0015010000000000902 0.5 0.17920700000000003" rpy="-1.5707963267948966 1.9929409209450203e-46 1.5707963267948966" />
         <parent link="$(arg prefix)Rear_Panel" />
         <child link="$(arg prefix)Top_Weld_Plate" />
     </joint>
-    <joint name="Front_Weld_Plate_and_Top_Panel" type="fixed">
+    <joint name="$(arg prefix)Front_Weld_Plate_and_Top_Panel" type="fixed">
         <origin xyz="0.5770000000000001 -0.34879999999999994 0.0015000000000000568" rpy="1.5707963267948966 2.552890093070388e-31 0.0" />
         <parent link="$(arg prefix)Top_Panel" />
         <child link="$(arg prefix)Front_Weld_Plate" />
     </joint>
-    <joint name="Black_Plate_Exhaust_and_Top_Panel" type="fixed">
+    <joint name="$(arg prefix)Black_Plate_Exhaust_and_Top_Panel" type="fixed">
         <origin xyz="0.5770000000000001 0.34880000000000005 0.0015000000000000568" rpy="1.5707963267948966 2.552890093070388e-31 0.0" />
         <parent link="$(arg prefix)Top_Panel" />
         <child link="$(arg prefix)Back_Plate_Exhaust" />
     </joint>
-    <joint name="Side_Plate_Left_and_Top_Panel" type="fixed">
+    <joint name="$(arg prefix)Side_Plate_Left_and_Top_Panel" type="fixed">
         <origin xyz="0.5770000000000001 -0.34879999999999994 0.0" rpy="0.0 2.552890093070388e-31 0.0" />
         <parent link="$(arg prefix)Top_Panel" />
         <child link="$(arg prefix)Side_Plates_Left" />
     </joint>
-    <joint name="Side_Plate_Right_and_Top_Panel" type="fixed">
+    <joint name="$(arg prefix)Side_Plate_Right_and_Top_Panel" type="fixed">
         <origin xyz="-0.5770000000000001 -0.34879999999999994 0.0015000000000000568" rpy="3.141592653589793 -2.552890093070388e-31 3.141592653589793" />
         <parent link="$(arg prefix)Top_Panel" />
         <child link="$(arg prefix)Side_Plates_Right" />
     </joint>
-    <joint name="Chute_House_and_Top_Panel" type="fixed">
+    <joint name="$(arg prefix)Chute_House_and_Top_Panel" type="fixed">
         <origin xyz="0.5770000000000001 -0.34879999999999994 0.0015000000000000568" rpy="1.5707963267948966 2.552890093070388e-31 0.0" />
         <parent link="$(arg prefix)Top_Panel" />
         <child link="$(arg prefix)Chute_01" />
     </joint>
-    <joint name="Pedestal_and_Bottom_Box" type="fixed">
+    <joint name="$(arg prefix)Pedestal_and_Bottom_Box" type="fixed">
         <origin xyz="0.5770000000000001 0.0 0.0" rpy="1.5707963267948966 -0.0 0.0" />
         <parent link="$(arg prefix)Bottom_Box" />
         <child link="$(arg prefix)Pedestal" />
     </joint>
-    <joint name="Top_Panel_and_Bottom_Box" type="fixed">
+    <joint name="$(arg prefix)Top_Panel_and_Bottom_Box" type="fixed">
         <origin xyz="0.5770000000000001 0.349 0.97" rpy="0.0 -0.0 0.0" />
         <parent link="$(arg prefix)Bottom_Box" />
         <child link="$(arg prefix)Top_Panel" />
     </joint>
-    <joint name="Light_1_and_Top_Weld_Plate" type="fixed">
+    <joint name="$(arg prefix)Light_1_and_Top_Weld_Plate" type="fixed">
         <origin xyz="0.0 -0.08709829 0.7088370399999999" rpy="1.5707963267948966 1.5707963267948966 0" />
         <parent link="$(arg prefix)Top_Weld_Plate" />
         <child link="$(arg prefix)light_1" />
     </joint>
-    <joint name="Light_2_and_Top_Weld_Plate" type="fixed">
+    <joint name="$(arg prefix)Light_2_and_Top_Weld_Plate" type="fixed">
         <origin xyz="0.0 -0.08769323 0.45740296" rpy="-1.5707963267948966 1.5707963267948966 0" />
         <parent link="$(arg prefix)Top_Weld_Plate" />
         <child link="$(arg prefix)light_2" />
     </joint>
-    <joint name="Top_Camera_Frame_and_Bottom_Box" type="fixed">
+    <joint name="$(arg prefix)Top_Camera_Frame_and_Bottom_Box" type="fixed">
         <origin xyz="0.5770000000000001 0.349 0.0" rpy="3.141592653589793 -0.0 0.0" />
         <parent link="$(arg prefix)Bottom_Box" />
         <child link="$(arg prefix)Top_Camera_frame" />
     </joint>
-    <joint name="Letter_Trimmer_Holder_and_Mail_Spreader_Housing" type="fixed">
-        <origin xyz="0.23 -0.105 0.005" rpy="-1.5707963267948966 2.924579959513007e-31 -1.5707963267948966" />
+    <joint name="$(arg prefix)Letter_Trimmer_Holder_and_Mail_Spreader_Housing" type="fixed">
+        <origin xyz="0.075 -0.105 0.005" rpy="-1.5707963267948966 2.9245799595130017e-31 -1.5707963267948966" />
         <parent link="$(arg prefix)Mail_Spreader_Housing" />
         <child link="$(arg prefix)Letter_Trimmer_Holder" />
     </joint>
-    <joint name="Mail_Top_Plate_and_Mail_Spreader_Housing" type="fixed">
-        <origin xyz="0.23 -0.17449999999999988 0.0" rpy="1.5707963267948966 -2.924579959513007e-31 1.5707963267948966" />
+    <joint name="$(arg prefix)Mail_Top_Plate_and_Mail_Spreader_Housing" type="fixed">
+        <origin xyz="0.075 -0.17449999999999988 0.0" rpy="1.5707963267948966 -2.9245799595130017e-31 1.5707963267948966" />
         <parent link="$(arg prefix)Mail_Spreader_Housing" />
         <child link="$(arg prefix)Mail_Top_Plate" />
     </joint>
-    <joint name="Mail_Spreader_Housing_and_Chute" type="fixed">
+    <joint name="$(arg prefix)Mail_Spreader_Housing_and_Chute" type="fixed">
         <origin xyz="-0.26322 0.0 -0.0015000000000000002" rpy="3.141592653589793 1.5707963267948966 0" />
         <parent link="$(arg prefix)Chute_01" />
         <child link="$(arg prefix)Mail_Spreader_Housing" />
     </joint>
-    <joint name="Vib_Rack_Base_and_Vib_Rack_Baseplate" type="fixed">
+    <joint name="$(arg prefix)Vib_Rack_Base_and_Vib_Rack_Baseplate" type="fixed">
         <origin xyz="0.0 0.05 0.305" rpy="3.141592653589793 -0.0 2.5528900930846764e-31" />
         <parent link="$(arg prefix)Vibration_Rack_Baseplate" />
         <child link="$(arg prefix)Vibration_Rack_Base" />
     </joint>
-    <joint name="Vib_Rack_and_Vib_Rack_Base" type="fixed">
+    <joint name="$(arg prefix)Vib_Rack_and_Vib_Rack_Base" type="fixed">
         <origin xyz="-0.23050000000000004 -0.03 0.155" rpy="0.0 -0.0 7.770197939968213e-32" />
         <parent link="$(arg prefix)Vibration_Rack_Base" />
         <child link="$(arg prefix)Vibration_Rack" />
     </joint>
-    <joint name="Vib_Rack_Baseplate_and_Top_Panel" type="fixed">
+    <joint name="$(arg prefix)Vib_Rack_Baseplate_and_Top_Panel" type="fixed">
         <origin xyz="0.0 0.0 0.0015000000000000568" rpy="1.5707963267948966 2.552890093070388e-31 0.0" />
         <parent link="$(arg prefix)Top_Panel" />
