Commit message: updated with new models

File: urdf/downdraft.xacro (robot description, xacro)
@@ -1,4 +1,4 @@
 <?xml version='1.0' encoding='utf-8'?>
-<robot xmlns:xacro="http://www.ros.org/wiki/xacro">
+<robot name="Downdraft_with_Joints">
     <link name="$(arg prefix)Pedestal">
         <inertial>
@@ -21,64 +21,4 @@
         </collision>
     </link>
-    <link name="$(arg prefix)Chute_01">
-        <inertial>
-            <origin xyz="-0.08249380309602244 0.023602865373523515 -0.21954822946951677" rpy="0.0 -0.0 0.0" />
-            <mass value="0.4016200251973849" />
-            <inertia ixx="0.005361750452761271" iyy="0.007420254096579371" izz="0.0028299950399888196" ixy="-0.00042653413194027046" iyz="0.0006737716338254679" ixz="0.0008355434112971155" />
-        </inertial>
-        <visual name="Chute_01_visual">
-            <origin xyz="-0.13872000000000215 -4.263256414560601e-16 -0.17350000000000076" rpy="3.944304526105066e-31 -2.719513272350892e-16 -5.208585445482765e-15" />
-            <geometry>
-                <mesh filename="package://trossen_arm_description/meshes/downdraft/Chute_01.stl" scale="0.001 0.001 0.001" />
-            </geometry>
-            <material name="orange" />
-        </visual>
-        <collision name="Chute_01_collision">
-            <origin xyz="-0.13872000000000215 -4.263256414560601e-16 -0.17350000000000076" rpy="3.944304526105066e-31 -2.719513272350892e-16 -5.208585445482765e-15" />
-            <geometry>
-                <mesh filename="package://trossen_arm_description/meshes/downdraft/Chute_01.stl" scale="0.001 0.001 0.001" />
-            </geometry>
-        </collision>
-    </link>
-    <link name="$(arg prefix)Chute_02">
-        <inertial>
-            <origin xyz="-0.05139987365201762 -0.004954008441779365 5.329070518200751e-16" rpy="0.0 -0.0 0.0" />
-            <mass value="0.13589450417228027" />
-            <inertia ixx="0.0002510152481522282" iyy="0.0003438571436062132" izz="9.509060396239999e-05" ixy="2.795320396681289e-07" iyz="-2.712554575719088e-34" ixz="-3.469446951953614e-18" />
-        </inertial>
-        <visual name="Chute_02_visual">
-            <origin xyz="-0.022999999999995566 -0.009999999999996163 6.039613253960852e-16" rpy="-1.5707963267948961 1.5707963267948952 0" />
-            <geometry>
-                <mesh filename="package://trossen_arm_description/meshes/downdraft/Chute_02.stl" scale="0.001 0.001 0.001" />
-            </geometry>
-            <material name="orange" />
-        </visual>
-        <collision name="Chute_02_collision">
-            <origin xyz="-0.022999999999995566 -0.009999999999996163 6.039613253960852e-16" rpy="-1.5707963267948961 1.5707963267948952 0" />
-            <geometry>
-                <mesh filename="package://trossen_arm_description/meshes/downdraft/Chute_02.stl" scale="0.001 0.001 0.001" />
-            </geometry>
-        </collision>
-    </link>
-    <link name="$(arg prefix)Chute_03">
-        <inertial>
-            <origin xyz="2.1535183236665035e-09 0.051219203865357915 0.004954181407317978" rpy="0.0 -1.1570498455835856e-76 0.0" />
-            <mass value="0.08184450417228083" />
-            <inertia ixx="5.776613298766331e-05" iyy="5.4695778535993056e-05" izz="0.00011110755509355363" ixy="-2.775534541600249e-17" iyz="1.6839673550484314e-07" ixz="3.6872531278104992e-19" />
-        </inertial>
-        <visual name="Chute_03_visual">
-            <origin xyz="2.1535183236665035e-09 0.022999999999997415 8.429368314466501e-16" rpy="-4.976592143281927e-30 1.1050127114447813e-15 6.938013042892593e-15" />
-            <geometry>
-                <mesh filename="package://trossen_arm_description/meshes/downdraft/Chute_03.stl" scale="0.001 0.001 0.001" />
-            </geometry>
-            <material name="orange" />
-        </visual>
-        <collision name="Chute_03_collision">
-            <origin xyz="2.1535183236665035e-09 0.022999999999997415 8.429368314466501e-16" rpy="-4.976592143281927e-30 1.1050127114447813e-15 6.938013042892593e-15" />
-            <geometry>
-                <mesh filename="package://trossen_arm_description/meshes/downdraft/Chute_03.stl" scale="0.001 0.001 0.001" />
-            </geometry>
-        </collision>
-    </link>
     <link name="$(arg prefix)Back_Plate_Exhaust">
         <inertial>
@@ -92,5 +32,5 @@
                 <mesh filename="package://trossen_arm_description/meshes/downdraft/Back_Plate_Exhaust.stl" scale="0.001 0.001 0.001" />
             </geometry>
-            <material name="light_blue" />
+            <material name="light_grey" />
         </visual>
         <collision name="Back_Plate_Exhaust_collision">
@@ -112,5 +52,5 @@
                 <mesh filename="package://trossen_arm_description/meshes/downdraft/Rear_Panel.stl" scale="0.001 0.001 0.001" />
             </geometry>
-            <material name="light_blue" />
+            <material name="light_grey" />
         </visual>
         <collision name="Rear_Panel_collision">
@@ -132,5 +72,5 @@
                 <mesh filename="package://trossen_arm_description/meshes/downdraft/Top_Panel.stl" scale="0.001 0.001 0.001" />
             </geometry>
-            <material name="light_blue" />
+            <material name="light_grey" />
         </visual>
         <collision name="Top_Panel_collision">
@@ -152,5 +92,5 @@
                 <mesh filename="package://trossen_arm_description/meshes/downdraft/Top_Weld_Plate.stl" scale="0.001 0.001 0.001" />
             </geometry>
-            <material name="light_blue" />
+            <material name="light_grey" />
         </visual>
         <collision name="Top_Weld_Plate_collision">
@@ -172,5 +112,5 @@
                 <mesh filename="package://trossen_arm_description/meshes/downdraft/Front_Weld_Plate.stl" scale="0.001 0.001 0.001" />
             </geometry>
-            <material name="light_blue" />
+            <material name="light_grey" />
         </visual>
         <collision name="Front_Weld_Plate_collision">
@@ -192,5 +132,5 @@
                 <mesh filename="package://trossen_arm_description/meshes/downdraft/Side_Plates_Left.stl" scale="0.001 0.001 0.001" />
             </geometry>
-            <material name="light_blue" />
+            <material name="light_grey" />
         </visual>
         <collision name="Side_Plates_Left_collision">
@@ -212,5 +152,5 @@
                 <mesh filename="package://trossen_arm_description/meshes/downdraft/Side_Plates_Right.stl" scale="0.001 0.001 0.001" />
             </geometry>
-            <material name="light_blue" />
+            <material name="light_grey" />
         </visual>
         <collision name="Side_Plates_Right_collision">
@@ -281,92 +221,12 @@
         </collision>
     </link>
-    <link name="$(arg prefix)Top_Camera_frame">
-        <inertial>
-            <origin xyz="0.0 -4.973799150320702e-16 -1.1161829652996849" rpy="0.0 -0.0 0.0" />
-            <mass value="522.5745" />
-            <inertia ixx="204.28774916813882" iyy="333.6312468650135" izz="172.02041519687438" ixy="-1.7053025658242404e-13" iyz="3.410605131648481e-13" ixz="0.0" />
-        </inertial>
-        <visual name="Top_Camera_frame_visual">
-            <origin xyz="-0.5769999999999998 0.3500000000000001 -2.842170943040401e-16" rpy="3.141592653589793 -0.0 0.0" />
-            <geometry>
-                <mesh filename="package://trossen_arm_description/meshes/downdraft/Top_Camera_frame.stl" scale="0.001 0.001 0.001" />
-            </geometry>
-            <material name="light_grey" />
-        </visual>
-        <collision name="Top_Camera_frame_collision">
-            <origin xyz="-0.5769999999999998 0.3500000000000001 -2.842170943040401e-16" rpy="3.141592653589793 -0.0 0.0" />
-            <geometry>
-                <mesh filename="package://trossen_arm_description/meshes/downdraft/Top_Camera_frame.stl" scale="0.001 0.001 0.001" />
-            </geometry>
-        </collision>
-    </link>
-    <link name="$(arg prefix)Mail_Spreader_Housing">
-        <inertial>
-            <origin xyz="0.2297487853588787 -0.09297671857199007 0.07359079941501165" rpy="0.0 -4.663963129396153e-77 0.0" />
-            <mass value="0.7818877668805357" />
-            <inertia ixx="0.003421827232823249" iyy="0.004391842901898424" izz="0.0033633324964867928" ixy="-8.893594203029931e-07" iyz="2.2033683713118535e-06" ixz="-9.834189106466829e-06" />
-        </inertial>
-        <visual name="Mail_Spreader_Housing_visual">
-            <origin xyz="0.23000000000000104 -0.10000000000000085 0.07500000000000015" rpy="-3.141592653589793 -1.5707963267948915 0" />
-            <geometry>
-                <mesh filename="package://trossen_arm_description/meshes/downdraft/Mail_Spreader_Housing.stl" scale="0.001 0.001 0.001" />
-            </geometry>
-            <material name="light_green" />
-        </visual>
-        <collision name="Mail_Spreader_Housing_collision">
-            <origin xyz="0.23000000000000104 -0.10000000000000085 0.07500000000000015" rpy="-3.141592653589793 -1.5707963267948915 0" />
-            <geometry>
-                <mesh filename="package://trossen_arm_description/meshes/downdraft/Mail_Spreader_Housing.stl" scale="0.001 0.001 0.001" />
-            </geometry>
-        </collision>
-    </link>
-    <link name="$(arg prefix)Mail_Top_Plate">
-        <inertial>
-            <origin xyz="3.258106006185813e-05 0.07820551417803287 1.0658141036401502e-15" rpy="-2.8486550277461034e-64 -0.0 0.0" />
-            <mass value="0.08915200000000002" />
-            <inertia ixx="0.0003873164201692175" iyy="0.0002032497645628878" izz="0.00018581264713210532" ixy="-1.370908783160374e-06" iyz="1.3738562485522464e-35" ixz="1.4022694188954473e-36" />
-        </inertial>
-        <visual name="Mail_Top_Plate_visual">
-            <origin xyz="-2.842170943040401e-16 0.07499999999999986 1.0302869668521452e-15" rpy="-3.141592653589793 -4.857225732735152e-16 -1.5707963267948915" />
-            <geometry>
-                <mesh filename="package://trossen_arm_description/meshes/downdraft/Mail_Top_Plate.stl" scale="0.001 0.001 0.001" />
-            </geometry>
-            <material name="light_green" />
-        </visual>
-        <collision name="Mail_Top_Plate_collision">
-            <origin xyz="-2.842170943040401e-16 0.07499999999999986 1.0302869668521452e-15" rpy="-3.141592653589793 -4.857225732735152e-16 -1.5707963267948915" />
-            <geometry>
-                <mesh filename="package://trossen_arm_description/meshes/downdraft/Mail_Top_Plate.stl" scale="0.001 0.001 0.001" />
-            </geometry>
-        </collision>
-    </link>
-    <link name="$(arg prefix)Letter_Trimmer_Holder">
-        <inertial>
-            <origin xyz="0.028766362717210114 -0.019520905574119354 -1.7763568394002506e-16" rpy="2.8486550277461034e-64 -0.0 0.0" />
-            <mass value="0.041840657300680255" />
-            <inertia ixx="4.5702849910761456e-05" iyy="7.059497852655167e-05" izz="3.356023542885889e-05" ixy="-2.2850515949621175e-06" iyz="-1.734723475976807e-18" ixz="-1.734723475976807e-18" />
-        </inertial>
-        <visual name="Letter_Trimmer_Holder_visual">
-            <origin xyz="0.034500000000000454 -0.0280000000000004 1.1723955140041654e-15" rpy="5.208585445482766e-15 -1.5707963267948961 0" />
-            <geometry>
-                <mesh filename="package://trossen_arm_description/meshes/downdraft/Letter_Trimmer_Holder.stl" scale="0.001 0.001 0.001" />
-            </geometry>
-            <material name="pink" />
-        </visual>
-        <collision name="Letter_Trimmer_Holder_collision">
-            <origin xyz="0.034500000000000454 -0.0280000000000004 1.1723955140041654e-15" rpy="5.208585445482766e-15 -1.5707963267948961 0" />
-            <geometry>
-                <mesh filename="package://trossen_arm_description/meshes/downdraft/Letter_Trimmer_Holder.stl" scale="0.001 0.001 0.001" />
-            </geometry>
-        </collision>
-    </link>
     <link name="$(arg prefix)Vibration_Rack">
         <inertial>
-            <origin xyz="-3.560925775730084e-05 -0.05658320071581926 0.03505806254969656" rpy="0.0 -0.0 0.0" />
+            <origin xyz="-3.560925775367707e-05 -0.056583200715837875 0.0350580625496977" rpy="0.0 -0.0 0.0" />
             <mass value="9.687032297505903" />
-            <inertia ixx="0.10672472798451338" iyy="0.3070441039085452" izz="0.23522193770247846" ixy="3.995602255724151e-06" iyz="0.003855536422117556" ixz="-1.2093209676544703e-05" />
+            <inertia ixx="0.10672472798451871" iyy="0.307044103908545" izz="0.23522193770248023" ixy="3.995602257056419e-06" iyz="0.003855536422118" ixz="-1.2093209676655725e-05" />
         </inertial>
         <visual name="Vibration_Rack_visual">
-            <origin xyz="-2.842170943040401e-16 7.389644451905042e-15 7.105427357601002e-17" rpy="-3.141592653589793 2.0907912740951003e-14 -2.7316076737125388e-14" />
+            <origin xyz="3.339550858072471e-15 -1.1226575225009583e-14 1.2079226507921704e-15" rpy="-3.141592653589793 2.0724215721078897e-14 -2.7316076737125385e-14" />
             <geometry>
                 <mesh filename="package://trossen_arm_description/meshes/downdraft/Vibration_Rack.stl" scale="0.001 0.001 0.001" />
@@ -375,5 +235,5 @@
         </visual>
         <collision name="Vibration_Rack_collision">
-            <origin xyz="-2.842170943040401e-16 7.389644451905042e-15 7.105427357601002e-17" rpy="-3.141592653589793 2.0907912740951003e-14 -2.7316076737125388e-14" />
+            <origin xyz="3.339550858072471e-15 -1.1226575225009583e-14 1.2079226507921704e-15" rpy="-3.141592653589793 2.0724215721078897e-14 -2.7316076737125385e-14" />
             <geometry>
                 <mesh filename="package://trossen_arm_description/meshes/downdraft/Vibration_Rack.stl" scale="0.001 0.001 0.001" />
@@ -383,17 +243,17 @@
     <link name="$(arg prefix)Vibration_Rack_Baseplate">
         <inertial>
-            <origin xyz="-0.23049999999999743 0.0059425450065914735 0.1499999999999993" rpy="0.0 -0.0 0.0" />
+            <origin xyz="-0.3460000000000062 -0.005942545006610232 -0.19700000000000187" rpy="0.0 -0.0 0.0" />
             <mass value="1.9339628174588095" />
-            <inertia ixx="0.02085303052106169" iyy="0.06366362420799082" izz="0.04294565651272153" ixy="-1.3322676295501878e-15" iyz="5.551115123125783e-17" ixz="-2.7755575615628914e-17" />
+            <inertia ixx="0.020853030521061244" iyy="0.06366362420799082" izz="0.042945656512721087" ixy="-1.2212453270876722e-15" iyz="0.0" ixz="0.0" />
         </inertial>
         <visual name="Vibration_Rack_Baseplate_visual">
-            <origin xyz="-0.23049999999999876 -6.8212102632969615e-15 0.1499999999999994" rpy="3.944304526105065e-31 1.6434924467491004e-15 2.960591172541443e-14" />
+            <origin xyz="-0.34600000000000486 -1.1795009413617664e-14 -0.19700000000000178" rpy="6.138323918751008e-30 1.8271894666212035e-15 -3.141592653589764" />
             <geometry>
                 <mesh filename="package://trossen_arm_description/meshes/downdraft/Vibration_Rack_Baseplate.stl" scale="0.001 0.001 0.001" />
             </geometry>
-            <material name="yellow" />
+            <material name="blue_green" />
         </visual>
         <collision name="Vibration_Rack_Baseplate_collision">
-            <origin xyz="-0.23049999999999876 -6.8212102632969615e-15 0.1499999999999994" rpy="3.944304526105065e-31 1.6434924467491004e-15 2.960591172541443e-14" />
+            <origin xyz="-0.34600000000000486 -1.1795009413617664e-14 -0.19700000000000178" rpy="6.138323918751008e-30 1.8271894666212035e-15 -3.141592653589764" />
             <geometry>
                 <mesh filename="package://trossen_arm_description/meshes/downdraft/Vibration_Rack_Baseplate.stl" scale="0.001 0.001 0.001" />
@@ -403,119 +263,209 @@
     <link name="$(arg prefix)Vibration_Rack_Base">
         <inertial>
-            <origin xyz="-0.23050000000000437 -0.025968639122598773 0.15500000000000866" rpy="0.0 -0.0 0.0" />
+            <origin xyz="-0.23050000000000068 -0.025968639122617532 0.15500000000000985" rpy="0.0 -0.0 0.0" />
             <mass value="1.7818591516603366" />
-            <inertia ixx="0.021644302791165693" iyy="0.06399137638580299" izz="0.04245645563593259" ixy="4.107825191113079e-15" iyz="-8.326672684688674e-16" ixz="1.7541523789077473e-14" />
+            <inertia ixx="0.021644302791166137" iyy="0.06399137638580299" izz="0.04245645563593259" ixy="4.107825191113079e-15" iyz="-8.881784197001252e-16" ixz="1.752764600126966e-14" />
         </inertial>
         <visual name="Vibration_Rack_Base_visual">
-            <origin xyz="-0.2304999999999872 -0.01999999999999204 0.15500000000000067" rpy="3.141592653589793 -6.998028758169689e-16 -2.855865576422289e-14" />
+            <origin xyz="-0.2304999999999835 -0.02000000000001066 0.15500000000000186" rpy="3.141592653589793 -8.834998956890721e-16 -2.855865576422289e-14" />
             <geometry>
                 <mesh filename="package://trossen_arm_description/meshes/downdraft/Vibration_Rack_Base.stl" scale="0.001 0.001 0.001" />
             </geometry>
+            <material name="blue_green" />
+        </visual>
+        <collision name="Vibration_Rack_Base_collision">
+            <origin xyz="-0.2304999999999835 -0.02000000000001066 0.15500000000000186" rpy="3.141592653589793 -8.834998956890721e-16 -2.855865576422289e-14" />
+            <geometry>
+                <mesh filename="package://trossen_arm_description/meshes/downdraft/Vibration_Rack_Base.stl" scale="0.001 0.001 0.001" />
+            </geometry>
+        </collision>
+    </link>
+    <link name="$(arg prefix)Chute_01">
+        <inertial>
+            <origin xyz="-0.15923825529236482 0.017829265726551285 -0.20976434579271125" rpy="0.0 -0.0 0.0" />
+            <mass value="1.1197714721887138" />
+            <inertia ixx="0.013536819321686044" iyy="0.019209838060771256" izz="0.0072772651963624035" ixy="0.0010343827538852324" iyz="0.0015588032150294917" ixz="-0.002556598061301485" />
+        </inertial>
+        <visual name="Chute_01_visual">
+            <origin xyz="-0.13700000000000473 -8.526512829121202e-16 -0.17650000000000138" rpy="2.6812065273393026e-31 1.5541371939922871e-15 -2.637781665533484e-15" />
+            <geometry>
+                <mesh filename="package://trossen_arm_description/meshes/downdraft/Chute_01.stl" scale="0.001 0.001 0.001" />
+            </geometry>
+            <material name="orange" />
+        </visual>
+        <collision name="Chute_01_collision">
+            <origin xyz="-0.13700000000000473 -8.526512829121202e-16 -0.17650000000000138" rpy="2.6812065273393026e-31 1.5541371939922871e-15 -2.637781665533484e-15" />
+            <geometry>
+                <mesh filename="package://trossen_arm_description/meshes/downdraft/Chute_01.stl" scale="0.001 0.001 0.001" />
+            </geometry>
+        </collision>
+    </link>
+    <link name="$(arg prefix)Mail_trimmer_Housing">
+        <inertial>
+            <origin xyz="0.2231330931020773 -0.07390510447320253 0.0824281580506026" rpy="0.0 -0.0 0.0" />
+            <mass value="2.446539063446293" />
+            <inertia ixx="0.012553930163533344" iyy="0.032292650030558256" izz="0.029256029100468428" ixy="-0.00017732766123468302" iyz="-0.00039022576504210704" ixz="-0.00021220463644744392" />
+        </inertial>
+        <visual name="Mail_trimmer_Housing_visual">
+            <origin xyz="0.22500000000000112 -0.09999999999999971 0.0850000000000044" rpy="3.141592653589793 -1.570796326794894 0" />
+            <geometry>
+                <mesh filename="package://trossen_arm_description/meshes/downdraft/Mail_trimmer_Housing.stl" scale="0.001 0.001 0.001" />
+            </geometry>
             <material name="green" />
         </visual>
-        <collision name="Vibration_Rack_Base_collision">
-            <origin xyz="-0.2304999999999872 -0.01999999999999204 0.15500000000000067" rpy="3.141592653589793 -6.998028758169689e-16 -2.855865576422289e-14" />
-            <geometry>
-                <mesh filename="package://trossen_arm_description/meshes/downdraft/Vibration_Rack_Base.stl" scale="0.001 0.001 0.001" />
-            </geometry>
-        </collision>
-    </link>
-    <joint name="Chute_Right_and_Chute_House" type="fixed">
-        <origin xyz="-0.26322 0.0019999999999998864 -0.17350000000000002" rpy="3.141592653589793 -2.465190328815662e-32 -1.5707963267948966" />
-        <parent link="$(arg prefix)Chute_01" />
-        <child link="$(arg prefix)Chute_02" />
-    </joint>
-    <joint name="Chute_Front_and_Chute_House" type="fixed">
-        <origin xyz="-0.0864698 0.0019999999999998864 -0.0015000000000000002" rpy="-3.141592653589793 1.3670076544845265e-15 -3.141592653589793" />
-        <parent link="$(arg prefix)Chute_01" />
-        <child link="$(arg prefix)Chute_03" />
-    </joint>
-    <joint name="Rear_Panel_and_Top_Panel" type="fixed">
+        <collision name="Mail_trimmer_Housing_collision">
+            <origin xyz="0.22500000000000112 -0.09999999999999971 0.0850000000000044" rpy="3.141592653589793 -1.570796326794894 0" />
+            <geometry>
+                <mesh filename="package://trossen_arm_description/meshes/downdraft/Mail_trimmer_Housing.stl" scale="0.001 0.001 0.001" />
+            </geometry>
+        </collision>
+    </link>
+    <link name="$(arg prefix)Mail_Trim_Cover">
+        <inertial>
+            <origin xyz="0.000133566473353568 -0.06008416612141275 0.15455947407350315" rpy="0.0 -0.0 0.0" />
+            <mass value="0.1640406666666669" />
+            <inertia ixx="0.0017024970182741017" iyy="0.0013707385195750599" izz="0.0003347270475937969" ixy="-1.4794741078072438e-06" iyz="-6.042398613870931e-05" ixz="-2.1896581987868036e-07" />
+        </inertial>
+        <visual name="Mail_Trim_Cover_visual">
+            <origin xyz="-5.684341886080802e-16 -0.0550000000000037 0.15000000000000102" rpy="-3.141592653589793 -8.084034387609881e-16 1.5707963267948952" />
+            <geometry>
+                <mesh filename="package://trossen_arm_description/meshes/downdraft/Mail_Trim_Cover.stl" scale="0.001 0.001 0.001" />
+            </geometry>
+            <material name="green" />
+        </visual>
+        <collision name="Mail_Trim_Cover_collision">
+            <origin xyz="-5.684341886080802e-16 -0.0550000000000037 0.15000000000000102" rpy="-3.141592653589793 -8.084034387609881e-16 1.5707963267948952" />
+            <geometry>
+                <mesh filename="package://trossen_arm_description/meshes/downdraft/Mail_Trim_Cover.stl" scale="0.001 0.001 0.001" />
+            </geometry>
+        </collision>
+    </link>
+    <link name="$(arg prefix)RealSense_Holder_01">
+        <inertial>
+            <origin xyz="-0.018229927806950458 -2.842170943040401e-16 0.004819089911902808" rpy="0.0 -0.0 0.0" />
+            <mass value="0.022472041856292764" />
+            <inertia ixx="7.987660902548932e-06" iyy="5.853876976928685e-06" izz="6.244287812387506e-06" ixy="1.4303025446890157e-39" iyz="8.673617379884035e-19" ixz="-2.2713681345834513e-07" />
+        </inertial>
+        <visual name="RealSense_Holder_01_visual">
+            <origin xyz="-0.015000000000005969 -2.842170943040401e-16 0.005499999999999403" rpy="5.551115123125783e-17 -1.5707963267948952 0" />
+            <geometry>
+                <mesh filename="package://trossen_arm_description/meshes/downdraft/RealSense_Holder_01.stl" scale="0.001 0.001 0.001" />
+            </geometry>
+            <material name="trossen_black" />
+        </visual>
+        <collision name="RealSense_Holder_01_collision">
+            <origin xyz="-0.015000000000005969 -2.842170943040401e-16 0.005499999999999403" rpy="5.551115123125783e-17 -1.5707963267948952 0" />
+            <geometry>
+                <mesh filename="package://trossen_arm_description/meshes/downdraft/RealSense_Holder_01.stl" scale="0.001 0.001 0.001" />
+            </geometry>
+        </collision>
+    </link>
+    <link name="$(arg prefix)RealSense_Holder_02">
+        <inertial>
+            <origin xyz="-0.005936392109073836 0.012500000000000497 -0.04390711772369166" rpy="0.0 -0.0 0.0" />
+            <mass value="0.04528239081499246" />
+            <inertia ixx="4.348175418397715e-05" iyy="3.834049476281187e-05" izz="7.948625230042028e-06" ixy="6.938893903907228e-18" iyz="-1.734723475976807e-18" ixz="2.096282809456451e-06" />
+        </inertial>
+        <visual name="RealSense_Holder_02_visual">
+            <origin xyz="-5.968558980384841e-15 0.012500000000000497 -0.05000000000000029" rpy="1.5707963267948968 1.2246467991473596e-16 -1.5707963267948981" />
+            <geometry>
+                <mesh filename="package://trossen_arm_description/meshes/downdraft/RealSense_Holder_02.stl" scale="0.001 0.001 0.001" />
+            </geometry>
+            <material name="trossen_black" />
+        </visual>
+        <collision name="RealSense_Holder_02_collision">
+            <origin xyz="-5.968558980384841e-15 0.012500000000000497 -0.05000000000000029" rpy="1.5707963267948968 1.2246467991473596e-16 -1.5707963267948981" />
+            <geometry>
+                <mesh filename="package://trossen_arm_description/meshes/downdraft/RealSense_Holder_02.stl" scale="0.001 0.001 0.001" />
+            </geometry>
+        </collision>
+    </link>
+    <joint name="$(arg prefix)Rear_Panel_and_Top_Panel" type="fixed">
         <origin xyz="0.5770000000000001 0.34880000000000005 0.0015000000000000568" rpy="1.5707963267948966 2.552890093070388e-31 0.0" />
         <parent link="$(arg prefix)Top_Panel" />
         <child link="$(arg prefix)Rear_Panel" />
     </joint>
-    <joint name="Top_Weld_Plate_and_Rear_Panel" type="fixed">
+    <joint name="$(arg prefix)Top_Weld_Plate_and_Rear_Panel" type="fixed">
         <origin xyz="-0.0015010000000000902 0.5 0.17920700000000003" rpy="-1.5707963267948966 1.9929409209450203e-46 1.5707963267948966" />
         <parent link="$(arg prefix)Rear_Panel" />
         <child link="$(arg prefix)Top_Weld_Plate" />
     </joint>
-    <joint name="Front_Weld_Plate_and_Top_Panel" type="fixed">
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