Commit message: new_model

File: urdf/downdraft.xacro (robot description, xacro)
@@ -3,10 +3,10 @@
     <link name="$(arg prefix)Pedestal">
         <inertial>
-            <origin xyz="2.486899575160351e-15 0.3075696855589309 0.24999999999999856" rpy="0.0 -0.0 0.0" />
+            <origin xyz="2.5579538487363606e-15 0.3075696855589309 0.3499999999999974" rpy="0.0 -0.0 0.0" />
             <mass value="589.894824375" />
-            <inertia ixx="34.27470062751247" iyy="15.58909217825311" izz="41.01537044013878" ixy="1.8474111129762605e-12" iyz="1.2079226507921703e-12" ixz="-2.8421709430404007e-13" />
+            <inertia ixx="34.27470062751246" iyy="15.589092178253225" izz="41.01537044013884" ixy="1.8616219676914625e-12" iyz="1.2079226507921703e-12" ixz="-2.984279490192421e-13" />
         </inertial>
         <visual name="Pedestal_visual">
-            <origin xyz="-0.5749999999999887 7.041719095097274e-17 0.09999999999999964" rpy="4.3367040406321e-15 1.2879808064022797e-15 -1.224646799147377e-16" />
+            <origin xyz="-0.5749999999999886 7.04171909509728e-17 0.19999999999999854" rpy="4.3367040406321e-15 1.2879808064022797e-15 -1.224646799147377e-16" />
             <geometry>
                 <mesh filename="package://trossen_arm_description/meshes/downdraft/Pedestal.stl" scale="0.001 0.001 0.001" />
@@ -15,67 +15,7 @@
         </visual>
         <collision name="Pedestal_collision">
-            <origin xyz="-0.5749999999999887 7.041719095097274e-17 0.09999999999999964" rpy="4.3367040406321e-15 1.2879808064022797e-15 -1.224646799147377e-16" />
+            <origin xyz="-0.5749999999999886 7.04171909509728e-17 0.19999999999999854" rpy="4.3367040406321e-15 1.2879808064022797e-15 -1.224646799147377e-16" />
             <geometry>
                 <mesh filename="package://trossen_arm_description/meshes/downdraft/Pedestal.stl" scale="0.001 0.001 0.001" />
-            </geometry>
-        </collision>
-    </link>
-    <link name="$(arg prefix)Chute_01">
-        <inertial>
-            <origin xyz="-0.08249380309602244 0.023602865373523515 -0.21954822946951677" rpy="0.0 -0.0 0.0" />
-            <mass value="0.4016200251973849" />
-            <inertia ixx="0.005361750452761271" iyy="0.007420254096579371" izz="0.0028299950399888196" ixy="-0.00042653413194027046" iyz="0.0006737716338254679" ixz="0.0008355434112971155" />
-        </inertial>
-        <visual name="Chute_01_visual">
-            <origin xyz="-0.13872000000000215 -4.263256414560601e-16 -0.17350000000000076" rpy="3.944304526105066e-31 -2.719513272350892e-16 -5.208585445482765e-15" />
-            <geometry>
-                <mesh filename="package://trossen_arm_description/meshes/downdraft/Chute_01.stl" scale="0.001 0.001 0.001" />
-            </geometry>
-            <material name="orange" />
-        </visual>
-        <collision name="Chute_01_collision">
-            <origin xyz="-0.13872000000000215 -4.263256414560601e-16 -0.17350000000000076" rpy="3.944304526105066e-31 -2.719513272350892e-16 -5.208585445482765e-15" />
-            <geometry>
-                <mesh filename="package://trossen_arm_description/meshes/downdraft/Chute_01.stl" scale="0.001 0.001 0.001" />
-            </geometry>
-        </collision>
-    </link>
-    <link name="$(arg prefix)Chute_02">
-        <inertial>
-            <origin xyz="-0.05139987365201762 -0.004954008441779365 5.329070518200751e-16" rpy="0.0 -0.0 0.0" />
-            <mass value="0.13589450417228027" />
-            <inertia ixx="0.0002510152481522282" iyy="0.0003438571436062132" izz="9.509060396239999e-05" ixy="2.795320396681289e-07" iyz="-2.712554575719088e-34" ixz="-3.469446951953614e-18" />
-        </inertial>
-        <visual name="Chute_02_visual">
-            <origin xyz="-0.022999999999995566 -0.009999999999996163 6.039613253960852e-16" rpy="-1.5707963267948961 1.5707963267948952 0" />
-            <geometry>
-                <mesh filename="package://trossen_arm_description/meshes/downdraft/Chute_02.stl" scale="0.001 0.001 0.001" />
-            </geometry>
-            <material name="orange" />
-        </visual>
-        <collision name="Chute_02_collision">
-            <origin xyz="-0.022999999999995566 -0.009999999999996163 6.039613253960852e-16" rpy="-1.5707963267948961 1.5707963267948952 0" />
-            <geometry>
-                <mesh filename="package://trossen_arm_description/meshes/downdraft/Chute_02.stl" scale="0.001 0.001 0.001" />
-            </geometry>
-        </collision>
-    </link>
-    <link name="$(arg prefix)Chute_03">
-        <inertial>
-            <origin xyz="2.1535183236665035e-09 0.051219203865357915 0.004954181407317978" rpy="0.0 -1.1570498455835856e-76 0.0" />
-            <mass value="0.08184450417228083" />
-            <inertia ixx="5.776613298766331e-05" iyy="5.4695778535993056e-05" izz="0.00011110755509355363" ixy="-2.775534541600249e-17" iyz="1.6839673550484314e-07" ixz="3.6872531278104992e-19" />
-        </inertial>
-        <visual name="Chute_03_visual">
-            <origin xyz="2.1535183236665035e-09 0.022999999999997415 8.429368314466501e-16" rpy="-4.976592143281927e-30 1.1050127114447813e-15 6.938013042892593e-15" />
-            <geometry>
-                <mesh filename="package://trossen_arm_description/meshes/downdraft/Chute_03.stl" scale="0.001 0.001 0.001" />
-            </geometry>
-            <material name="orange" />
-        </visual>
-        <collision name="Chute_03_collision">
-            <origin xyz="2.1535183236665035e-09 0.022999999999997415 8.429368314466501e-16" rpy="-4.976592143281927e-30 1.1050127114447813e-15 6.938013042892593e-15" />
-            <geometry>
-                <mesh filename="package://trossen_arm_description/meshes/downdraft/Chute_03.stl" scale="0.001 0.001 0.001" />
             </geometry>
         </collision>
@@ -281,81 +221,101 @@
         </collision>
     </link>
-    <link name="$(arg prefix)Top_Camera_frame">
-        <inertial>
-            <origin xyz="0.0 -4.973799150320702e-16 -1.1161829652996849" rpy="0.0 -0.0 0.0" />
-            <mass value="522.5745" />
-            <inertia ixx="204.28774916813882" iyy="333.6312468650135" izz="172.02041519687438" ixy="-1.7053025658242404e-13" iyz="3.410605131648481e-13" ixz="0.0" />
-        </inertial>
-        <visual name="Top_Camera_frame_visual">
-            <origin xyz="-0.5769999999999998 0.3500000000000001 -2.842170943040401e-16" rpy="3.141592653589793 -0.0 0.0" />
-            <geometry>
-                <mesh filename="package://trossen_arm_description/meshes/downdraft/Top_Camera_frame.stl" scale="0.001 0.001 0.001" />
-            </geometry>
-            <material name="light_grey" />
-        </visual>
-        <collision name="Top_Camera_frame_collision">
-            <origin xyz="-0.5769999999999998 0.3500000000000001 -2.842170943040401e-16" rpy="3.141592653589793 -0.0 0.0" />
-            <geometry>
-                <mesh filename="package://trossen_arm_description/meshes/downdraft/Top_Camera_frame.stl" scale="0.001 0.001 0.001" />
-            </geometry>
-        </collision>
-    </link>
-    <link name="$(arg prefix)Mail_Spreader_Housing">
-        <inertial>
-            <origin xyz="0.2297487853588787 -0.09297671857199007 0.07359079941501165" rpy="0.0 -4.663963129396153e-77 0.0" />
-            <mass value="0.7818877668805357" />
-            <inertia ixx="0.003421827232823249" iyy="0.004391842901898424" izz="0.0033633324964867928" ixy="-8.893594203029931e-07" iyz="2.2033683713118535e-06" ixz="-9.834189106466829e-06" />
-        </inertial>
-        <visual name="Mail_Spreader_Housing_visual">
-            <origin xyz="0.23000000000000104 -0.10000000000000085 0.07500000000000015" rpy="-3.141592653589793 -1.5707963267948915 0" />
-            <geometry>
-                <mesh filename="package://trossen_arm_description/meshes/downdraft/Mail_Spreader_Housing.stl" scale="0.001 0.001 0.001" />
+    <link name="$(arg prefix)Chute_01">
+        <inertial>
+            <origin xyz="-0.17973825529236506 0.017829265726551 -0.21026434579271083" rpy="0.0 -0.0 0.0" />
+            <mass value="1.1197714721887138" />
+            <inertia ixx="0.013536819321686044" iyy="0.019209838060771034" izz="0.007277265196361515" ixy="0.0010343827538852324" iyz="0.0015588032150294362" ixz="-0.002556598061301485" />
+        </inertial>
+        <visual name="Chute_01_visual">
+            <origin xyz="-0.15750000000000497 -1.1368683772161603e-15 -0.17700000000000096" rpy="3.9443045261050538e-31 1.5541371939922844e-15 -2.637781665533484e-15" />
+            <geometry>
+                <mesh filename="package://trossen_arm_description/meshes/downdraft/Chute_01.stl" scale="0.001 0.001 0.001" />
+            </geometry>
+            <material name="orange" />
+        </visual>
+        <collision name="Chute_01_collision">
+            <origin xyz="-0.15750000000000497 -1.1368683772161603e-15 -0.17700000000000096" rpy="3.9443045261050538e-31 1.5541371939922844e-15 -2.637781665533484e-15" />
+            <geometry>
+                <mesh filename="package://trossen_arm_description/meshes/downdraft/Chute_01.stl" scale="0.001 0.001 0.001" />
+            </geometry>
+        </collision>
+    </link>
+    <link name="$(arg prefix)Mail_trimmer_Housing">
+        <inertial>
+            <origin xyz="0.19513309310207694 -0.07390510447320167 0.07242815805060261" rpy="0.0 -0.0 0.0" />
+            <mass value="2.446539063446293" />
+            <inertia ixx="0.012553930163532456" iyy="0.032292650030558034" izz="0.029256029100468872" ixy="-0.00017732766123468302" iyz="-0.00039022576504166295" ixz="-0.00021220463644744392" />
+        </inertial>
+        <visual name="Mail_trimmer_Housing_visual">
+            <origin xyz="0.19700000000000073 -0.09999999999999887 0.07500000000000441" rpy="3.141592653589793 -1.570796326794894 0" />
+            <geometry>
+                <mesh filename="package://trossen_arm_description/meshes/downdraft/Mail_trimmer_Housing.stl" scale="0.001 0.001 0.001" />
             </geometry>
             <material name="light_green" />
         </visual>
-        <collision name="Mail_Spreader_Housing_collision">
-            <origin xyz="0.23000000000000104 -0.10000000000000085 0.07500000000000015" rpy="-3.141592653589793 -1.5707963267948915 0" />
-            <geometry>
-                <mesh filename="package://trossen_arm_description/meshes/downdraft/Mail_Spreader_Housing.stl" scale="0.001 0.001 0.001" />
-            </geometry>
-        </collision>
-    </link>
-    <link name="$(arg prefix)Mail_Top_Plate">
-        <inertial>
-            <origin xyz="3.258106006185813e-05 0.07820551417803287 1.0658141036401502e-15" rpy="-2.8486550277461034e-64 -0.0 0.0" />
-            <mass value="0.08915200000000002" />
-            <inertia ixx="0.0003873164201692175" iyy="0.0002032497645628878" izz="0.00018581264713210532" ixy="-1.370908783160374e-06" iyz="1.3738562485522464e-35" ixz="1.4022694188954473e-36" />
-        </inertial>
-        <visual name="Mail_Top_Plate_visual">
-            <origin xyz="-2.842170943040401e-16 0.07499999999999986 1.0302869668521452e-15" rpy="-3.141592653589793 -4.857225732735152e-16 -1.5707963267948915" />
-            <geometry>
-                <mesh filename="package://trossen_arm_description/meshes/downdraft/Mail_Top_Plate.stl" scale="0.001 0.001 0.001" />
+        <collision name="Mail_trimmer_Housing_collision">
+            <origin xyz="0.19700000000000073 -0.09999999999999887 0.07500000000000441" rpy="3.141592653589793 -1.570796326794894 0" />
+            <geometry>
+                <mesh filename="package://trossen_arm_description/meshes/downdraft/Mail_trimmer_Housing.stl" scale="0.001 0.001 0.001" />
+            </geometry>
+        </collision>
+    </link>
+    <link name="$(arg prefix)Mail_Trim_Cover">
+        <inertial>
+            <origin xyz="0.00013356647335299954 -0.06008416612141375 0.1545594740735028" rpy="0.0 -0.0 0.0" />
+            <mass value="0.1640406666666669" />
+            <inertia ixx="0.0017024970182741017" iyy="0.0013707385195751154" izz="0.0003347270475937969" ixy="-1.4794741077794882e-06" iyz="-6.042398613870584e-05" ixz="-2.1896581988561925e-07" />
+        </inertial>
+        <visual name="Mail_Trim_Cover_visual">
+            <origin xyz="-1.1368683772161603e-15 -0.05500000000000469 0.1500000000000007" rpy="-3.141592653589793 -8.084034387609863e-16 1.5707963267948952" />
+            <geometry>
+                <mesh filename="package://trossen_arm_description/meshes/downdraft/Mail_Trim_Cover.stl" scale="0.001 0.001 0.001" />
             </geometry>
             <material name="light_green" />
         </visual>
-        <collision name="Mail_Top_Plate_collision">
-            <origin xyz="-2.842170943040401e-16 0.07499999999999986 1.0302869668521452e-15" rpy="-3.141592653589793 -4.857225732735152e-16 -1.5707963267948915" />
-            <geometry>
-                <mesh filename="package://trossen_arm_description/meshes/downdraft/Mail_Top_Plate.stl" scale="0.001 0.001 0.001" />
-            </geometry>
-        </collision>
-    </link>
-    <link name="$(arg prefix)Letter_Trimmer_Holder">
-        <inertial>
-            <origin xyz="0.028766362717210114 -0.019520905574119354 -1.7763568394002506e-16" rpy="2.8486550277461034e-64 -0.0 0.0" />
-            <mass value="0.041840657300680255" />
-            <inertia ixx="4.5702849910761456e-05" iyy="7.059497852655167e-05" izz="3.356023542885889e-05" ixy="-2.2850515949621175e-06" iyz="-1.734723475976807e-18" ixz="-1.734723475976807e-18" />
-        </inertial>
-        <visual name="Letter_Trimmer_Holder_visual">
-            <origin xyz="0.034500000000000454 -0.0280000000000004 1.1723955140041654e-15" rpy="5.208585445482766e-15 -1.5707963267948961 0" />
-            <geometry>
-                <mesh filename="package://trossen_arm_description/meshes/downdraft/Letter_Trimmer_Holder.stl" scale="0.001 0.001 0.001" />
+        <collision name="Mail_Trim_Cover_collision">
+            <origin xyz="-1.1368683772161603e-15 -0.05500000000000469 0.1500000000000007" rpy="-3.141592653589793 -8.084034387609863e-16 1.5707963267948952" />
+            <geometry>
+                <mesh filename="package://trossen_arm_description/meshes/downdraft/Mail_Trim_Cover.stl" scale="0.001 0.001 0.001" />
+            </geometry>
+        </collision>
+    </link>
+    <link name="$(arg prefix)Vibration_Rack_Baseplate">
+        <inertial>
+            <origin xyz="-0.2310000000000106 -0.007944669402224918 -0.20550000000000157" rpy="0.0 -0.0 0.0" />
+            <mass value="0.6190328174588098" />
+            <inertia ixx="0.010079775557782056" iyy="0.01517000847085618" izz="0.005196081105983352" ixy="-2.775557561562892e-17" iyz="-1.3877787807814457e-17" ixz="1.0408340855860843e-17" />
+        </inertial>
+        <visual name="Vibration_Rack_Baseplate_visual">
+            <origin xyz="-0.2310000000000058 -1.9895196601282807e-15 -0.2055000000000016" rpy="3.96682110745274e-31 1.4316725140775477e-15 -3.141592653589793" />
+            <geometry>
+                <mesh filename="package://trossen_arm_description/meshes/downdraft/Vibration_Rack_Baseplate.stl" scale="0.001 0.001 0.001" />
             </geometry>
             <material name="pink" />
         </visual>
-        <collision name="Letter_Trimmer_Holder_collision">
-            <origin xyz="0.034500000000000454 -0.0280000000000004 1.1723955140041654e-15" rpy="5.208585445482766e-15 -1.5707963267948961 0" />
-            <geometry>
-                <mesh filename="package://trossen_arm_description/meshes/downdraft/Letter_Trimmer_Holder.stl" scale="0.001 0.001 0.001" />
+        <collision name="Vibration_Rack_Baseplate_collision">
+            <origin xyz="-0.2310000000000058 -1.9895196601282807e-15 -0.2055000000000016" rpy="3.96682110745274e-31 1.4316725140775477e-15 -3.141592653589793" />
+            <geometry>
+                <mesh filename="package://trossen_arm_description/meshes/downdraft/Vibration_Rack_Baseplate.stl" scale="0.001 0.001 0.001" />
+            </geometry>
+        </collision>
+    </link>
+    <link name="$(arg prefix)Vibration_Rack_Base">
+        <inertial>
+            <origin xyz="-0.10591324987236309 0.027639411551972727 -0.159629420493331" rpy="0.0 -0.0 0.0" />
+            <mass value="0.9520007627842192" />
+            <inertia ixx="0.011957110018708361" iyy="0.0179409417489461" izz="0.006070444107805217" ixy="1.353927494285312e-07" iyz="1.3587317603536153e-06" ixz="4.862940201702526e-07" />
+        </inertial>
+        <visual name="Vibration_Rack_Base_visual">
+            <origin xyz="-0.10599999999999409 0.021000000000001934 -0.1605000000000016" rpy="2.833821430729822e-31 1.4316725140775477e-15 6.12323399573679e-17" />
+            <geometry>
+                <mesh filename="package://trossen_arm_description/meshes/downdraft/Vibration_Rack_Base.stl" scale="0.001 0.001 0.001" />
+            </geometry>
+            <material name="pink" />
+        </visual>
+        <collision name="Vibration_Rack_Base_collision">
+            <origin xyz="-0.10599999999999409 0.021000000000001934 -0.1605000000000016" rpy="2.833821430729822e-31 1.4316725140775477e-15 6.12323399573679e-17" />
+            <geometry>
+                <mesh filename="package://trossen_arm_description/meshes/downdraft/Vibration_Rack_Base.stl" scale="0.001 0.001 0.001" />
             </geometry>
         </collision>
@@ -363,17 +323,17 @@
     <link name="$(arg prefix)Vibration_Rack">
         <inertial>
-            <origin xyz="-3.560925775730084e-05 -0.05658320071581926 0.03505806254969656" rpy="0.0 -0.0 0.0" />
-            <mass value="9.687032297505903" />
-            <inertia ixx="0.10672472798451338" iyy="0.3070441039085452" izz="0.23522193770247846" ixy="3.995602255724151e-06" iyz="0.003855536422117556" ixz="-1.2093209676544703e-05" />
+            <origin xyz="-0.12049999999989904 -0.05942951406682354 0.20839735358378417" rpy="0.0 -0.0 0.0" />
+            <mass value="4.868368242409034" />
+            <inertia ixx="0.052860547298390514" iyy="0.068176771161919" izz="0.034347774077427395" ixy="-1.3322676295501878e-14" iyz="0.0016408924015689497" ixz="-1.609823385706477e-14" />
         </inertial>
         <visual name="Vibration_Rack_visual">
-            <origin xyz="-2.842170943040401e-16 7.389644451905042e-15 7.105427357601002e-17" rpy="-3.141592653589793 2.0907912740951003e-14 -2.7316076737125388e-14" />
+            <origin xyz="-0.12049999999997912 -1.7053025658242404e-15 0.1749999999999866" rpy="-3.141592653589793 -1.3704401741201799e-15 -1.2246467991473557e-16" />
             <geometry>
                 <mesh filename="package://trossen_arm_description/meshes/downdraft/Vibration_Rack.stl" scale="0.001 0.001 0.001" />
             </geometry>
-            <material name="blue_green" />
+            <material name="pink" />
         </visual>
         <collision name="Vibration_Rack_collision">
-            <origin xyz="-2.842170943040401e-16 7.389644451905042e-15 7.105427357601002e-17" rpy="-3.141592653589793 2.0907912740951003e-14 -2.7316076737125388e-14" />
+            <origin xyz="-0.12049999999997912 -1.7053025658242404e-15 0.1749999999999866" rpy="-3.141592653589793 -1.3704401741201799e-15 -1.2246467991473557e-16" />
             <geometry>
                 <mesh filename="package://trossen_arm_description/meshes/downdraft/Vibration_Rack.stl" scale="0.001 0.001 0.001" />
@@ -381,141 +341,81 @@
         </collision>
     </link>
-    <link name="$(arg prefix)Vibration_Rack_Baseplate">
-        <inertial>
-            <origin xyz="-0.23049999999999743 0.0059425450065914735 0.1499999999999993" rpy="0.0 -0.0 0.0" />
-            <mass value="1.9339628174588095" />
-            <inertia ixx="0.02085303052106169" iyy="0.06366362420799082" izz="0.04294565651272153" ixy="-1.3322676295501878e-15" iyz="5.551115123125783e-17" ixz="-2.7755575615628914e-17" />
-        </inertial>
-        <visual name="Vibration_Rack_Baseplate_visual">
-            <origin xyz="-0.23049999999999876 -6.8212102632969615e-15 0.1499999999999994" rpy="3.944304526105065e-31 1.6434924467491004e-15 2.960591172541443e-14" />
-            <geometry>
-                <mesh filename="package://trossen_arm_description/meshes/downdraft/Vibration_Rack_Baseplate.stl" scale="0.001 0.001 0.001" />
-            </geometry>
-            <material name="yellow" />
-        </visual>
-        <collision name="Vibration_Rack_Baseplate_collision">
-            <origin xyz="-0.23049999999999876 -6.8212102632969615e-15 0.1499999999999994" rpy="3.944304526105065e-31 1.6434924467491004e-15 2.960591172541443e-14" />
-            <geometry>
-                <mesh filename="package://trossen_arm_description/meshes/downdraft/Vibration_Rack_Baseplate.stl" scale="0.001 0.001 0.001" />
-            </geometry>
-        </collision>
-    </link>
-    <link name="$(arg prefix)Vibration_Rack_Base">
-        <inertial>
-            <origin xyz="-0.23050000000000437 -0.025968639122598773 0.15500000000000866" rpy="0.0 -0.0 0.0" />
-            <mass value="1.7818591516603366" />
-            <inertia ixx="0.021644302791165693" iyy="0.06399137638580299" izz="0.04245645563593259" ixy="4.107825191113079e-15" iyz="-8.326672684688674e-16" ixz="1.7541523789077473e-14" />
-        </inertial>
-        <visual name="Vibration_Rack_Base_visual">
-            <origin xyz="-0.2304999999999872 -0.01999999999999204 0.15500000000000067" rpy="3.141592653589793 -6.998028758169689e-16 -2.855865576422289e-14" />
-            <geometry>
-                <mesh filename="package://trossen_arm_description/meshes/downdraft/Vibration_Rack_Base.stl" scale="0.001 0.001 0.001" />
-            </geometry>
-            <material name="green" />
-        </visual>
-        <collision name="Vibration_Rack_Base_collision">
-            <origin xyz="-0.2304999999999872 -0.01999999999999204 0.15500000000000067" rpy="3.141592653589793 -6.998028758169689e-16 -2.855865576422289e-14" />
-            <geometry>
-                <mesh filename="package://trossen_arm_description/meshes/downdraft/Vibration_Rack_Base.stl" scale="0.001 0.001 0.001" />
-            </geometry>
-        </collision>
-    </link>
-    <joint name="Chute_Right_and_Chute_House" type="fixed">
-        <origin xyz="-0.26322 0.0019999999999998864 -0.17350000000000002" rpy="3.141592653589793 -2.465190328815662e-32 -1.5707963267948966" />
-        <parent link="$(arg prefix)Chute_01" />
-        <child link="$(arg prefix)Chute_02" />
-    </joint>
-    <joint name="Chute_Front_and_Chute_House" type="fixed">
-        <origin xyz="-0.0864698 0.0019999999999998864 -0.0015000000000000002" rpy="-3.141592653589793 1.3670076544845265e-15 -3.141592653589793" />
-        <parent link="$(arg prefix)Chute_01" />
-        <child link="$(arg prefix)Chute_03" />
-    </joint>
-    <joint name="Rear_Panel_and_Top_Panel" type="fixed">
+    <joint name="$(arg prefix)Rear_Panel_and_Top_Panel" type="fixed">
         <origin xyz="0.5770000000000001 0.34880000000000005 0.0015000000000000568" rpy="1.5707963267948966 2.552890093070388e-31 0.0" />
         <parent link="$(arg prefix)Top_Panel" />
         <child link="$(arg prefix)Rear_Panel" />
     </joint>
-    <joint name="Top_Weld_Plate_and_Rear_Panel" type="fixed">
+    <joint name="$(arg prefix)Top_Weld_Plate_and_Rear_Panel" type="fixed">
         <origin xyz="-0.0015010000000000902 0.5 0.17920700000000003" rpy="-1.5707963267948966 1.9929409209450203e-46 1.5707963267948966" />
         <parent link="$(arg prefix)Rear_Panel" />
         <child link="$(arg prefix)Top_Weld_Plate" />
     </joint>
-    <joint name="Front_Weld_Plate_and_Top_Panel" type="fixed">
+    <joint name="$(arg prefix)Front_Weld_Plate_and_Top_Panel" type="fixed">
         <origin xyz="0.5770000000000001 -0.34879999999999994 0.0015000000000000568" rpy="1.5707963267948966 2.552890093070388e-31 0.0" />
         <parent link="$(arg prefix)Top_Panel" />
         <child link="$(arg prefix)Front_Weld_Plate" />
     </joint>
-    <joint name="Black_Plate_Exhaust_and_Top_Panel" type="fixed">
+    <joint name="$(arg prefix)Back_Plate_Exhaust_and_Top_Panel" type="fixed">
         <origin xyz="0.5770000000000001 0.34880000000000005 0.0015000000000000568" rpy="1.5707963267948966 2.552890093070388e-31 0.0" />
         <parent link="$(arg prefix)Top_Panel" />
         <child link="$(arg prefix)Back_Plate_Exhaust" />
     </joint>
-    <joint name="Side_Plate_Left_and_Top_Panel" type="fixed">
+    <joint name="$(arg prefix)Side_Plate_Left_and_Top_Panel" type="fixed">
         <origin xyz="0.5770000000000001 -0.34879999999999994 0.0" rpy="0.0 2.552890093070388e-31 0.0" />
         <parent link="$(arg prefix)Top_Panel" />
         <child link="$(arg prefix)Side_Plates_Left" />
     </joint>
-    <joint name="Side_Plate_Right_and_Top_Panel" type="fixed">
+    <joint name="$(arg prefix)Side_Plate_Right_and_Top_Panel" type="fixed">
         <origin xyz="-0.5770000000000001 -0.34879999999999994 0.0015000000000000568" rpy="3.141592653589793 -2.552890093070388e-31 3.141592653589793" />
         <parent link="$(arg prefix)Top_Panel" />
         <child link="$(arg prefix)Side_Plates_Right" />
     </joint>
-    <joint name="Chute_House_and_Top_Panel" type="fixed">
-        <origin xyz="0.5770000000000001 -0.34879999999999994 0.0015000000000000568" rpy="1.5707963267948966 2.552890093070388e-31 0.0" />
-        <parent link="$(arg prefix)Top_Panel" />
-        <child link="$(arg prefix)Chute_01" />
-    </joint>
-    <joint name="Pedestal_and_Bottom_Box" type="fixed">
+    <joint name="$(arg prefix)Pedestal_and_Bottom_Box" type="fixed">
         <origin xyz="0.5770000000000001 0.0 0.0" rpy="1.5707963267948966 -0.0 0.0" />
         <parent link="$(arg prefix)Bottom_Box" />
         <child link="$(arg prefix)Pedestal" />
     </joint>
-    <joint name="Top_Panel_and_Bottom_Box" type="fixed">
+    <joint name="$(arg prefix)Top_Panel_and_Bottom_Box" type="fixed">
         <origin xyz="0.5770000000000001 0.349 0.97" rpy="0.0 -0.0 0.0" />
         <parent link="$(arg prefix)Bottom_Box" />
         <child link="$(arg prefix)Top_Panel" />
     </joint>
-    <joint name="Light_1_and_Top_Weld_Plate" type="fixed">
+    <joint name="$(arg prefix)Light_1_and_Top_Weld_Plate" type="fixed">
         <origin xyz="0.0 -0.08709829 0.7088370399999999" rpy="1.5707963267948966 1.5707963267948966 0" />
         <parent link="$(arg prefix)Top_Weld_Plate" />
         <child link="$(arg prefix)light_1" />
     </joint>
-    <joint name="Light_2_and_Top_Weld_Plate" type="fixed">
+    <joint name="$(arg prefix)Light_2_and_Top_Weld_Plate" type="fixed">
         <origin xyz="0.0 -0.08769323 0.45740296" rpy="-1.5707963267948966 1.5707963267948966 0" />
         <parent link="$(arg prefix)Top_Weld_Plate" />
         <child link="$(arg prefix)light_2" />
     </joint>
-    <joint name="Top_Camera_Frame_and_Bottom_Box" type="fixed">
-        <origin xyz="0.5770000000000001 0.349 0.0" rpy="3.141592653589793 -0.0 0.0" />
-        <parent link="$(arg prefix)Bottom_Box" />
-        <child link="$(arg prefix)Top_Camera_frame" />
-    </joint>
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